File: KiCAD/Main/MCU.kicad_sch (KiCad schematic)
At the start: 26 parts, among them Q4 2N7002, SW1 RESET, SW2 USER, U4 STM32H750VBTx, Y2 SiT8008xx-2x-xxE (25MHz)

Commit message: Complete layout first draft
Connections:
- net BMP390 (SPI4) CS1: now also U4.57 (PD10); no longer U4.55 (PD8)
- net BMP390 (SPI4) CS3: now also U4.55 (PD8); no longer U4.57 (PD10)
- net GPS_RESET: now also U4.86 (PD5); no longer U4.24 (PA2)
- net SIMU CS2: now also U4.97 (PE0); no longer U4.38 (PE8)
- net Servo1_DOut: now also U4.38 (PE8); no longer U4.82 (PD1)
- net Servo1_Encoder: now also U4.40 (PE10); no longer U4.84 (PD3)
- net Servo2_DOut: now also U4.39 (PE9); no longer U4.83 (PD2)
- net Servo2_Encoder: now also U4.41 (PE11); no longer U4.85 (PD4)
