File: KiCAD/Main/MCU.kicad_sch (KiCad schematic)
At the start: 26 parts, among them Q4 2N7002, SW1 RESET, SW2 USER, U4 STM32H750VBTx, Y2 SiT8008xx-2x-xxE (25MHz)

Commit message: It2 12-29-2025
Connections:
- net SIMU CS2: now also U4.96 (PB9); no longer U4.97 (PE0)
- net SIMU CS3: now also U4.97 (PE0); no longer U4.35 (PB1)
Changed lines of the file:
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@@
+		)
+	)
+	(hierarchical_label "SIMU CS3"
+		(shape output)
+		(at 78.74 64.77 180)
+		(effects
+			(font
+				(size 1.27 1.27)
+			)
+			(justify right)
 		)
 	)
@@
 		)
 	)
-	(hierarchical_label "SIMU CS3"
-		(shape output)
-		(at 124.46 87.63 0)
-		(effects
-			(font
-				(size 1.27 1.27)
-			)
-			(justify left)
-		)
-	)
 	(hierarchical_label "DEBUG_JTMS-SWCLK"
 		(shape input)
@@
 		)
 	)
+	(hierarchical_label "GPS SCL"
+		(shape output)
+		(at 78.74 138.43 180)
+		(effects
+			(font
+				(size 1.27 1.27)
+			)
+			(justify right)
+		)
+	)
+	(hierarchical_label "SD_Det"
+		(shape input)
+		(at 124.46 80.01 0)
+		(effects
+			(font
+				(size 1.27 1.27)
+			)
+			(justify left)
+		)
+	)
+	(hierarchical_label "SIMU CLK"
+		(shape output)
+		(at 124.46 92.71 0)
+		(effects
+			(font
+				(size 1.27 1.27)
+			)
+			(justify left)
+		)
+	)
 	(hierarchical_label "SIMU CS2"
 		(shape output)
-		(at 78.74 64.77 180)
-		(effects
-			(font
-				(size 1.27 1.27)
-			)
-			(justify right)
-		)
-	)
-	(hierarchical_label "GPS SCL"
-		(shape output)
-		(at 78.74 138.43 180)
-		(effects
-			(font
-				(size 1.27 1.27)
-			)
-			(justify right)
-		)
-	)
-	(hierarchical_label "SD_Det"
-		(shape input)
-		(at 124.46 80.01 0)
-		(effects
-			(font
-				(size 1.27 1.27)
-			)
-			(justify left)
-		)
-	)
-	(hierarchical_label "SIMU CLK"
-		(shape output)
-		(at 124.46 92.71 0)
-		(effects
-			(font
+		(at 124.46 107.95 0)
+		(effects
+			(font
