File: KiCAD/Main/Main.kicad_pcb (KiCad board)
At the start: 4 copper layers, 80.2 x 150 mm, 95 parts, among them J1 Micro_SD_Card_Det2, J2 Screw_Terminal_01x09, J3 Screw_Terminal_01x09, J4 USB_C_Receptacle_USB2.0_16P, J7 Conn_02x05_Top_Bottom_Mountin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, J8 Conn_Coaxial, J9 Conn_Coaxial, Q1 AO3400A, Q2 AO3400A, Q3 AO3400A, Q4 2N7002, SW1 RESET, SW2 USER, U1 LM2596S-3.3, U11 BMP390L, U12 BMP390L, U13 BMP390L, U14 BMI270, U15 BMI270, U16 BMI270, U17 SHT4x, U2 TPS2121RUXR, U3 BMM350, U4 STM32H750VBTx, U5 MAX-M8Q, U7 ISM6HG256x, U9 BME280, Y2 SiT8008xx-2x-xxE (25MHz)

Commit message: Complete layout first draft
Parts:
- removed U10: ~, E22-900T22S:E22-900T22S
- removed U9: BME280, Package_LGA:Bosch_LGA-8_2.5x2.5mm_P0.65mm_ClockwisePinNumbering
- added C17: 100n, Capacitor_SMD:C_0603_1608Metric, F.Cu at (101.5, 61.2)
- added C18: 10n, Capacitor_SMD:C_0603_1608Metric, F.Cu at (101.5, 63.0)
- added C19: 100n, Capacitor_SMD:C_0603_1608Metric, F.Cu at (106.5, 43.0)
- added R16: 10k, Resistor_SMD:R_0603_1608Metric, F.Cu at (106.5, 44.8)
- added U6: ~, E22-900T22S:E22-900T22S, F.Cu at (91.0, 51.0)
- moved JP2 77.9 mm to (85.7, 64.7)
- moved U15 59.6 mm to (81.0, 68.4)
- moved U14 58.5 mm to (74.0, 68.4)
- moved C33 58.2 mm to (86.5, 71.7)
- moved C34 58.2 mm to (89.5, 71.7)
- moved C30 58.2 mm to (79.5, 72.0)
- moved C32 58.2 mm to (82.5, 72.0)
- moved C29 58.1 mm to (72.5, 72.0)
- moved C31 58.1 mm to (75.5, 72.0)
- moved U16 57.7 mm to (88.0, 68.7)
- moved C23 54.9 mm to (119.2, 78.8)
- moved C24 54.3 mm to (117.8, 72.8)
- moved U3 53.9 mm to (116.2, 74.5), turned to 90 degrees
- moved C25 52.9 mm to (115.8, 78.8), turned to 90 degrees
- moved C22 43.4 mm to (119.2, 100.8), turned to -90 degrees
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Connections:
- C29 pad 1: Net-(U14-VDDIO) -> +3V3
- J7 pad 2: unconnected-(J7-Pin_2-Pad2) -> /SWCLK
- J7 pad 3: GND -> unconnected-(J7-Pin_3-Pad3)
- J7 pad 4: +3V3 -> /SWDIO
- J7 pad 5: Net-(D6-A) -> GND
- J7 pad 6: /Microcontroller/DEBUG_JTMS-SWCLK -> GND
- J7 pad 7: /Microcontroller/DEBUG_JTMS-SWDIO -> +3V3
- J7 pad 8: GND -> +3V3
- J7 pad 9: +3V3 -> Net-(D6-A)
- U14 pad 5: Net-(U14-VDDIO) -> +3V3
- U4 pad 24: /GPS/GPS_RESET -> unconnected-(U4-PA2-Pad24)
- U4 pad 38: /Microcontroller/SIMU CS2 -> /Microcontroller/Servo1_DOut
- U4 pad 39: unconnected-(U4-PE9-Pad39) -> /Microcontroller/Servo2_DOut
- U4 pad 40: unconnected-(U4-PE10-Pad40) -> /Microcontroller/Servo1_Encoder
- U4 pad 41: unconnected-(U4-PE11-Pad41) -> /Microcontroller/Servo2_Encoder
- U4 pad 55: /Barometer/BMP390_CS1 -> /Barometer/BMP390_CS3
- U4 pad 57: /Barometer/BMP390_CS3 -> /Barometer/BMP390_CS1
- U4 pad 72: /Microcontroller/DEBUG_JTMS-SWDIO -> /SWDIO
- U4 pad 76: /Microcontroller/DEBUG_JTMS-SWCLK -> /SWCLK
- U4 pad 82: /Microcontroller/Servo1_DOut -> unconnected-(U4-PD1-Pad82)
- U4 pad 83: /Microcontroller/Servo2_DOut -> unconnected-(U4-PD2-Pad83)
- U4 pad 84: /Microcontroller/Servo1_Encoder -> unconnected-(U4-PD3-Pad84)
- U4 pad 85: /Microcontroller/Servo2_Encoder -> unconnected-(U4-PD4-Pad85)
- U4 pad 86: unconnected-(U4-PD5-Pad86) -> /GPS/GPS_RESET
- U4 pad 97: unconnected-(U4-PE0-Pad97) -> /Microcontroller/SIMU CS2
- U7 pad 7: unconnected-(U7-GND-Pad7) -> GND
Routing:
- net Net-(D3-A): track 0.00 -> 229.0 mm, vias 0 -> 1
- net /Barometer/BMP390_MISO: track 0.00 -> 172.7 mm, vias 0 -> 5
- net /Barometer/BMP390_MOSI: track 0.00 -> 167.2 mm, vias 0 -> 4
- net /Microcontroller/SIMU MOSI: track 0.00 -> 121.9 mm, vias 0 -> 9
- net +3V3: track 60.7 -> 157.9 mm, vias 7 -> 28
- net GND: track 154.1 -> 238.3 mm, vias 14 -> 80
- net /Microcontroller/SIMU CLK: track 0.00 -> 80.7 mm, vias 0 -> 4
- net /Microcontroller/SIMU CS1: track 0.00 -> 77.7 mm
- net /Microcontroller/Servo1_DOut: track 0.00 -> 77.1 mm, vias 0 -> 1
- net /Microcontroller/SIMU1 INT: track 0.00 -> 74.7 mm, vias 0 -> 2
- net /Microcontroller/Main Eject: track 0.00 -> 74.2 mm, vias 0 -> 2
- net /Microcontroller/Servo2_DOut: track 0.00 -> 73.8 mm, vias 0 -> 1
- net /Microcontroller/Drogue Eject Backup: track 0.00 -> 72.2 mm, vias 0 -> 2
- net /Microcontroller/Servo1_Encoder: track 0.00 -> 71.0 mm, vias 0 -> 1
- net /GPS/GPS_RESET: track 0.00 -> 69.6 mm, vias 0 -> 4
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- added copper zone on In2.Cu, net +3V3
- added copper zone on In1.Cu, net GND
Other:
- board size 80.2 x 150 mm -> 61.8 x 150 mm
