File: KiCAD/Main/Main.kicad_pcb (KiCad board)
At the start: 4 copper layers, 60 x 150 mm, 95 parts, among them J1 Micro_SD_Card_Det2, J2 Screw_Terminal_01x09, J3 Screw_Terminal_01x09, J4 USB_C_Receptacle_USB2.0_16P, J5 Conn_02x04_Counter_Clockwise, J8 Conn_Coaxial, J9 Conn_Coaxial, Q1 AO3400A, Q2 AO3400A, Q3 AO3400A, Q4 2N7002, SW1 RESET, SW2 USER, U1 LM2596S-3.3, U11 BMP390L, U12 BMP390L, U13 BMP390L, U14 BMI270, U15 BMI270, U16 BMI270, U17 SHT4x, U2 TPS2121RUXR, U3 LIS2MDL, U4 STM32H750VBTx, U5 MAX-M8Q, U7 ISM6HG256x, Y2 SiT8008xx-2x-xxE (25MHz)

Commit message: Layout and routing
Parts:
- added H1: MountingHole, MountingHole:MountingHole_3.2mm_M3, F.Cu at (113.3, 70.0)
- added H2: MountingHole, MountingHole:MountingHole_3.2mm_M3, F.Cu at (152.4, 51.2)
- added H3: MountingHole, MountingHole:MountingHole_3.2mm_M3, F.Cu at (163.6, 175.9)
- added H4: MountingHole, MountingHole:MountingHole_3.2mm_M3, F.Cu at (112.4, 176.1)
- D2: moved to B.Cu
- JP2, JP3: footprint Jumper:SolderJumper-2_P1.3mm_Open_TrianglePad1.0x1.5mm -> Jumper:SolderJumper-2_P1.3mm_Open_RoundedPad1.0x1.5mm
- moved BZ1 34.7 mm to (157.8, 103.2)
- moved Q4 27.8 mm to (160.6, 110.3), turned to 180 degrees
- moved R12 27.4 mm to (163.3, 110.4)
- moved U1 25.1 mm to (124.9, 112.8), turned to 180 degrees
- moved C1 23.4 mm to (131.7, 119.3), turned to 0 degrees
- moved C15 19.3 mm to (141.1, 105.3), turned to 180 degrees
- moved L1 18.7 mm to (141.9, 110.3)
- moved C28 17.2 mm to (156.7, 85.6)
- moved U13 16.4 mm to (151.9, 87.3), turned to -90 degrees
- moved D2 15.2 mm to (141.9, 114.4)
- moved C27 14.5 mm to (156.7, 87.1)
- moved JP3 12.1 mm to (157.8, 83.3), turned to 0 degrees
- moved R2 11.0 mm to (111.7, 99.7), turned to 90 degrees
- moved C2 10.5 mm to (146.3, 114.3)
- moved R5 10.5 mm to (147.9, 114.3)
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Connections:
- U4 pad 3: /Microcontroller/Drogue Eject Main -> unconnected-(U4-PE4-Pad3)
- U4 pad 36: /Microcontroller/SIMU1 INT -> /Microcontroller/SIMU3 INT
- U4 pad 37: /Microcontroller/SIMU CS1 -> /Microcontroller/SIMU CS3
- U4 pad 4: /Microcontroller/Drogue Eject Backup -> unconnected-(U4-PE5-Pad4)
- U4 pad 40: /Microcontroller/SIMU3 INT -> /Microcontroller/SIMU1 INT
- U4 pad 41: /Microcontroller/SIMU CS3 -> /Microcontroller/SIMU CS1
- U4 pad 5: /Microcontroller/Main Eject -> unconnected-(U4-PE6-Pad5)
- U4 pad 61: unconnected-(U4-PD14-Pad61) -> /Microcontroller/USER_LED
- U4 pad 62: unconnected-(U4-PD15-Pad62) -> /Microcontroller/USER_BTN
- U4 pad 63: /Microcontroller/Servo1_DOut -> /Microcontroller/Servo2_DOut
- U4 pad 64: /Microcontroller/Servo2_DOut -> /Microcontroller/Servo1_DOut
- U4 pad 66: /Microcontroller/USER_LED -> /Microcontroller/Main Eject
- U4 pad 67: /Microcontroller/USER_BTN -> /Microcontroller/Drogue Eject Backup
- U4 pad 68: unconnected-(U4-PA9-Pad68) -> /Microcontroller/Drogue Eject Main
Routing:
- net /Microcontroller/Servo1_DOut: track 0.00 -> 132.3 mm, vias 0 -> 1
- net /Microcontroller/Servo2_DOut: track 0.00 -> 127.0 mm, vias 0 -> 1
- net /Microcontroller/Main Eject: track 0.00 -> 121.7 mm, vias 0 -> 2
- net /Microcontroller/Drogue Eject Backup: track 0.00 -> 117.6 mm, vias 0 -> 2
- net /Microcontroller/Drogue Eject Main: track 0.00 -> 114.3 mm, vias 0 -> 2
- net +3V3: track 0.00 -> 113.2 mm, vias 0 -> 35
- net GND: track 0.00 -> 95.6 mm, vias 0 -> 120
- net /Microcontroller/Servo1_Encoder: track 0.00 -> 92.1 mm, vias 0 -> 1
- net /Microcontroller/USER_BTN: track 0.00 -> 90.7 mm, vias 0 -> 2
- net /Microcontroller/Servo2_Encoder: track 0.00 -> 84.9 mm, vias 0 -> 1
- net /Microcontroller/USER_LED: track 0.00 -> 71.0 mm, vias 0 -> 2
- net /~{RESET}: track 0.00 -> 58.4 mm, vias 0 -> 1
- net /Microcontroller/BUZZER: track 0.00 -> 54.2 mm, vias 0 -> 2
- net +5V: track 0.00 -> 44.1 mm
- net Net-(D3-A): track 0.00 -> 43.1 mm
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- added copper zone on F.Cu, net Net-(D3-A)
Other:
- board text added: "BARO TMR"
- board text added: "RST"
- board text added: "SIMU TMR"
