File: KiCAD/Main/Main.kicad_sch (KiCad schematic)
At the start: 2 parts, among them J7 Conn_02x05_Top_Bottom_Mountin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

Commit message: It2 12-29-2025
Parts:
- J7: footprint Connector_IDC:IDC-Header_2x05_P2.54mm_Horizontal -> Connector_PinSocket_2.54mm:PinSocket_2x05_P2.54mm_Vertical
Changed lines of the file:
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@@
 			)
 		)
-		(property "Footprint" "Connector_IDC:IDC-Header_2x05_P2.54mm_Horizontal"
+		(property "Footprint" "Connector_PinSocket_2.54mm:PinSocket_2x05_P2.54mm_Vertical"
 			(at 53.34 95.25 0)
 			(effects
