File: KiCAD/Main/SIMUs.kicad_sch (KiCad schematic)
At the start: 10 parts, among them U14 BMI270, U15 BMI270, U16 BMI270

Commit message: Complete layout first draft
Connections:
- net +3V3: now also C29.1, U14.5 (VDDIO)
Changed lines of the file:
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@@
+	)
+	(junction
+		(at 175.26 29.21)
+		(diameter 0)
+		(color 0 0 0 0)
 	)
 	(junction
@@
 	(wire
 		(pts
+			(xy 175.26 29.21) (xy 186.69 29.21)
+		)
+		(stroke
+			(width 0)
+			(type default)
+		)
+	)
+	(wire
+		(pts
 			(xy 127 77.47) (xy 204.47 77.47)
 		)
@@
 		)
 		(stroke
+			(width 0)
+			(type default)
+		)
+	)
+	(wire
+		(pts
+			(xy 186.69 29.21) (xy 186.69 31.75)
+		)
+		(stroke
