File: KiCAD/Main/Power_Essentials.kicad_sch (KiCad schematic)
At the start: 26 parts, among them J1 Micro_SD_Card_Det2, J2 Screw_Terminal_01x09, J3 Screw_Terminal_01x09, J4 USB_C_Receptacle_USB2.0_16P, Q1 AO3400A, Q2 AO3400A, Q3 AO3400A, U1 LM2596S-3.3, U2 TPS2121RUXR

Commit message: Moved custom footprints into local KiCAD footprint library
Parts:
- U2: footprint TPS2121RUXR:IC_TPS2121RUXR -> Package_DFN_QFN:Texas_VQFN-HR-12_2x2.5mm_P0.5mm_ThermalVias
Changed lines of the file:
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@@
 			)
 		)
-		(property "Footprint" "TPS2121RUXR:IC_TPS2121RUXR"
+		(property "Footprint" "Package_DFN_QFN:Texas_VQFN-HR-12_2x2.5mm_P0.5mm_ThermalVias"
 			(at 194.31 54.61 0)
 			(effects
