File: KiCAD/Main/IMU_CTRLFRK/IMU_CTRLFRK.kicad_sch (KiCad schematic)
At the start: 13 parts, among them U3 LIS2MDL, U7 ISM6HG256x

Commit message: Reorganize libraries into LRI.pretty, replace BMI270 with BMI323
Parts:
- U7: footprint LRI:ISM6 -> LRI:ISM6HG256XTR
Changed lines of the file:
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@@
 			)
 		)
-		(property "Footprint" "LRI:ISM6"
+		(property "Footprint" "LRI:ISM6HG256XTR"
 			(at 110.49 104.14 0)
 			(effects
