File: KiCAD/Main/Barometric Altimeter/Barometric Altimeter.kicad_sch (KiCad schematic)
At the start: 7 parts, among them U11 BMP390L, U12 BMP390L, U13 BMP390L

Commit message: Layout and routing
Parts:
- JP3: footprint Jumper:SolderJumper-2_P1.3mm_Open_TrianglePad1.0x1.5mm -> Jumper:SolderJumper-2_P1.3mm_Open_RoundedPad1.0x1.5mm
Changed lines of the file:
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@@
 			)
 		)
-		(property "Footprint" "Jumper:SolderJumper-2_P1.3mm_Open_TrianglePad1.0x1.5mm"
+		(property "Footprint" "Jumper:SolderJumper-2_P1.3mm_Open_RoundedPad1.0x1.5mm"
 			(at 162.56 43.18 0)
 			(effects
