File: KiCAD/Soldering Practice Board/Main/BMI270.kicad_sch (KiCad schematic)
At the start: 1 part, among them U2 BMI160

Commit message: Complete BMI260 Explanation
Parts:
- added C1, C2: 100n, symbol Device:C
Connections:
- net +3V3: now also C1.1, C2.1
- net GND: now also C1.2, C2.2
Other:
- note added: "MOSI (Master Out Slave In). This corresponds to SDx, and according to the BMI260 datasheet is the data input for SPI. In I2C mode (See LIS2DH12) SDx is the data input and output, as the datasheet says."
- note added: "SCK (Sensor Clock) The clock pin establishes a constant stream of data, a simple square wave. This square wave is how the sensor times data input and output, synchronizing the operation and data input/output signals."
- note added: "These two capacitors are called decoupling capacitors. They smooth the voltage input into the sensor and ensure that no noise affects the voltage input. This is a safety measure, but a quite necessary one. The value of each capacitor is not always listed on the datasheets, so when in doubt, use 100n as the capacitance value. Connect the in parallel with sensor input voltages, and reference datash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"

Commit message: Configure IOC file, rename pins
Parts:
- C1, C2: footprint (none) -> Capacitor_SMD:C_0603_1608Metric
Changed lines of the file:
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@@
 			)
 		)
-		(property "Footprint" ""
+		(property "Footprint" "Capacitor_SMD:C_0603_1608Metric"
 			(at 194.6148 109.22 0)
 			(effects
@@
 			)
 		)
-		(property "Footprint" ""
+		(property "Footprint" "Capacitor_SMD:C_0603_1608Metric"
 			(at 200.3552 93.98 0)
 			(effects
