File: KiCAD/Soldering Practice Board/Main/Main.kicad_pcb (KiCad board)
At the start: 2 copper layers, 7 parts, among them U1 STM32C071R8Tx, U2 BMI160, U3 LSM6DS3

Commit message: begin stl pcb layout
Parts:
- moved U3 29.9 mm to (140.5, 70.0)
- moved C4 23.3 mm to (140.0, 75.0), turned to 90 degrees
- moved C3 19.3 mm to (146.0, 71.0)
- moved U1 3.68 mm to (140.0, 85.0)
Routing:
- net +3V3: track 0.00 -> 6.98 mm, vias 0 -> 2
- net GND: track 0.00 -> 2.53 mm, vias 0 -> 2
Changed lines of the file:
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@@
 	(footprint "Package_LGA:LGA-14_3x2.5mm_P0.5mm_LayoutBorder3x4y"
 		(layer "F.Cu")
-		(at 143.3375 99.75)
+		(at 140.5 70)
 		(descr "LGA, 14 Pin (https://www.st.com/resource/en/datasheet/lsm6ds3tr-c.pdf), generated with kicad-footprint-generator ipc_noLead_generator.py")
 		(tags "LGA NoLead")
@@
 	(footprint "Capacitor_SMD:C_0603_1608Metric"
 		(layer "F.Cu")
-		(at 160.225 86.5)
+		(at 140 75 90)
 		(descr "Capacitor SMD 0603 (1608 Metric), square (rectangular) end terminal, IPC-7351 nominal, (Body size source: IPC-SM-782 page 76, https://www.pcb-3d.com/wordpress/wp-content/uploads/ipc-sm-782a_amendment_1_and_2.pdf), generated with kicad-footprint-generator")
 		(tags "capacitor")
 		(property "Reference" "C4"
-			(at 0 -1.43 0)
+			(at 0 -1.5 90)
 			(layer "F.SilkS")
 			(effects
@@
 		)
 		(property "Value" "100n"
-			(at 0 1.43 0)
+			(at 0 1.43 90)
 			(layer "F.Fab")
 			(effects
@@
 		)
 		(property "Datasheet" "~"
-			(at 0 0 0)
+			(at 0 0 90)
 			(layer "F.Fab")
 			(hide yes)
@@
 		)
 		(property "Description" "Unpolarized capacitor"
-			(at 0 0 0)
+			(at 0 0 90)
 			(layer "F.Fab")
 			(hide yes)
@@
 		)
 		(fp_line
+			(start 1.48 -0.73)
+			(end 1.48 0.73)
+			(stroke
+				(width 0.05)
+				(type solid)
+			)
+			(layer "F.CrtYd")
+		)
+		(fp_line
 			(start -1.48 -0.73)
 			(end 1.48 -0.73)
@@
 		)
 		(fp_line
+			(start 1.48 0.73)
+			(end -1.48 0.73)
+			(stroke
+				(width 0.05)
+				(type solid)
+			)
+			(layer "F.CrtYd")
+		)
+		(fp_line
 			(start -1.48 0.73)
 			(end -1.48 -0.73)
@@
 		)
 		(fp_line
-			(start 1.48 -0.73)
-			(end 1.48 0.73)
-			(stroke
-				(width 0.05)
-				(type solid)
-			)
-			(layer "F.CrtYd")
-		)
-		(fp_line
-			(start 1.48 0.73)
-			(end -1.48 0.73)
-			(stroke
-				(width 0.05)
-				(type solid)
-			)
-			(layer "F.CrtYd")
+			(start 0.8 -0.4)
+			(end 0.8 0.4)
+			(stroke
+				(width 0.1)
+				(type solid)
+			)
+			(layer "F.Fab")
 		)
 		(fp_line
@@
 		)
 		(fp_line
+			(start 0.8 0.4)
+			(end -0.8 0.4)
+			(stroke
+				(width 0.1)
+				(type solid)
+			)
+			(layer "F.Fab")
+		)
+		(fp_line
 			(start -0.8 0.4)
 			(end -0.8 -0.4)
@@
 			(layer "F.Fab")
 		)
-		(fp_line
-			(start 0.8 -0.4)
-			(end 0.8 0.4)
-			(stroke
-				(width 0.1)
-				(type solid)
-			)
-			(layer "F.Fab")
-		)
-		(fp_line
-			(start 0.8 0.4)
-			(end -0.8 0.4)
-			(stroke
-				(width 0.1)
-				(type solid)
-			)
-			(layer "F.Fab")
-		)
 		(fp_text user "${REFERENCE}"
-			(at 0 0 0)
+			(at 0 0 90)
 			(layer "F.Fab")
 			(effects
@@
 		)
 		(pad "1" smd roundrect
-			(at -0.775 0)
+			(at -0.775 0 90)
 			(size 0.9 0.95)
 			(layers "F.Cu" "F.Mask" "F.Paste")
@@
 		)
 		(pad "2" smd roundrect
-			(at 0.775 0)
+			(at 0.775 0 90)
 			(size 0.9 0.95)
 			(layers "F.Cu" "F.Mask" "F.Paste")
@@
 	(footprint "Package_QFP:LQFP-64_10x10mm_P0.5mm"
 		(layer "F.Cu")
-		(at 141.3725 88.415)
+		(at 140 85)
 		(descr "LQFP, 64 Pin (https://www.analog.com/media/en/technical-documentation/data-sheets/ad7606_7606-6_7606-4.pdf), generated with kicad-footprint-generator ipc_gullwing_generator.py")
 		(tags "LQFP QFP")
@@
 	(footprint "Capacitor_SMD:C_0603_1608Metric"
 		(layer "F.Cu")
-		(at 160.225 83.99)
+		(at 146 71)
 		(descr "Capacitor SMD 0603 (1608 Metric), square (rectangular) end terminal, IPC-7351 nominal, (Body size source: IPC-SM-782 page 76, https://www.pcb-3d.com/wordpress/wp-content/uploads/ipc-sm-782a_amendment_1_and_2.pdf), generated with kicad-footprint-generator")
 		(tags "capacitor")
@@
 		)
 	)
+	(segment
+		(start 141.6625 70.75)
+		(end 144 70.75)
+		(width 0.2)
+		(layer "F.Cu")
+		(net 69)
+	)
+	(segment
+		(start 140 73)
+		(end 140 74.225)
+		(width 0.2)
+		(layer "F.Cu")
+		(net 69)
+	)
+	(segment
+		(start 144.975 70.75)
+		(end 145.225 71)
+		(width 0.2)
+		(layer "F.Cu")
+		(net 69)
+	)
+	(segment
+		(start 144 70.75)
+		(end 144.975 70.75)
+		(width 0.2)
+		(layer "F.Cu")
+		(net 69)
+	)
+	(segment
+		(start 140 70.9125)
+		(end 140 73)
+		(width 0.2)
+		(layer "F.Cu")
+		(net 69)
+	)
+	(via
+		(at 140 73)
+		(size 0.6)
+		(drill 0.3)
+		(layers "F.Cu" "B.Cu")
+		(net 69)
+	)
+	(via
+		(at 144 70.75)
+		(size 0.6)
+		(drill 0.3)
+		(layers "F.Cu" "B.Cu")
+		(net 69)
+	)
+	(segment
+		(start 140 75.775)
+		(end 139.725 75.775)
+		(width 0.2)
+		(layer "F.Cu")
+		(net 74)
+	)
+	(segment
+		(start 146.775 71)
+		(end 148 71)
+		(width 0.2)
+		(layer "F.Cu")
+		(net 74)
+	)
+	(segment
+		(start 139.725 75.775)
+		(end 139 76.5)
+		(width 0.2)
+		(layer "F.Cu")
+		(net 74)
+	)
+	(via
+		(at 139 76.5)
+		(size 0.6)
+		(drill 0.3)
+		(layers "F.Cu" "B.Cu")
+		(net 74)
+	)
+	(via
+		(at 148 71)
+		(size 0.6)
+		(drill 0.3)
+		(layers "F.Cu" "B.Cu")
+		(net 74)
+	)
 	(embedded_fonts no)
